File: arduino/busylight_schematic.kicad_sch (KiCad schematic)
At the start: 30 parts, among them J0 LED TREE, J1 RS-485, J2 To pin of J0, J3 Conn_01x01_Socket, J4 Conn_01x01_Socket, J5 Conn_01x01_Socket, U0 ULN2003A, U1 THVD1439

Commit message: wip
Parts:
- removed J1: RS-485, symbol Connector:Screw_Terminal_01x06
- removed J3, J4, J5: Conn_01x01_Socket, symbol Connector:Conn_01x01_Socket
- removed R_{x}0, R_{x}1, R_{x}2, R_{x}3, R_{x}4, R_{x}5, R_{x}6, R_{x}7: R*, symbol Device:R_US
- added J1: RS-485, symbol Connector:Screw_Terminal_01x16
- added Rx0*, Rx1*: R_Network04, Resistor_THT:R_Array_SIP5, symbol Device:R_Network04
Connections:
- net Earth: now also J1.13 (Pin_13), J1.14 (Pin_14), J1.7 (Pin_7), J1.8 (Pin_8)
- net at D_{x}1.1 (K): now also Rx0*.4 (R3)
- net at J2.1 (Pin_1): now also Rx0*.1 (common), Rx1*.1 (common)
- net at D_{x}4.1 (K): now also Rx1*.5 (R4)
- net at D_{x}3.1 (K): now also Rx0*.2 (R1)
- net at D_{x}5.1 (K): now also Rx1*.4 (R3)
- net at D_{x}7.1 (K): now also Rx1*.2 (R1)
- net at D_{x}0.1 (K): now also Rx0*.5 (R4)
- net at D_{x}2.1 (K): now also Rx0*.3 (R2)
- net at D_{x}6.1 (K): now also Rx1*.3 (R2)
- net at A0.24 (RAW): now also J1.15 (Pin_15), J1.16 (Pin_16)
- net at U1.6 (A): now also J1.11 (Pin_11), J1.9 (Pin_9)
- net at U1.7 (B): now also J1.10 (Pin_10), J1.12 (Pin_12)
- new net: J1.1 (Pin_1), J1.2 (Pin_2)
- new net: J1.3 (Pin_3), J1.4 (Pin_4)
- new net: J1.5 (Pin_5), J1.6 (Pin_6)
Other:
- note added: "8-PIN CAT6 CABLES A (IN) AND B (OUT)"
- note added: "A1 RDATA A(+) IN"
- note added: "A2 RDATA B(-) IN"
- note added: "A3 CC+ IN / +9V POWER SUPPLY"
- note added: "A4 DATA B(-) IN"
- note added: "A5 DATA A(+) IN"
- note added: "A6 CCr IN"
- note added: "A7 GND"
- note added: "A8 GND"
- note added: "B1 RDATA A(+) OUT"
- note added: "B2 RDATA B(-) OUT"
- note added: "B3 CC+ OUT"
- note added: "B4 DATA B(-) OUT"
- note added: "B5 DATA A(+) OUT"
- note added: "B6 CCr OUT"
- note added: "B7 GND"
- note added: "B8 GND"
- note added: "Powered via USB connector on Pro Micro board or external supply on "RAW" (which runs through the internal 5V regulator on the Pro Micro)."
- note removed: "+5V"
- note removed: "+Vin 6-12V"
- note removed: "A IN"
- note removed: "A OUT"
- note removed: "B IN"
- note removed: "B OUT"
- note removed: "GND"
- note removed: "Power Connections (Wired to Board)"
- note removed: "Powered via USB connector on Pro Micro board or external regulated supply on Vcc. Direct control over USB connector to host."
- moved on the sheet: D_{x}0, D_{x}1, D_{x}3, D_{x}5, D_{x}6, D_{x}7, R_{term}
